Commit message: added cameras in xarm

File: xarm_ros_code/xarm_ros/xarm_description/urdf/camera/camera.gazebo.xacro (robot description, xacro)
@@ -25,6 +25,8 @@
     </link>
     <joint name="${prefix}joint_camera" type="fixed">
-      <origin xyz="0.692 0.001 1.17" rpy="0 1.5708 0" />
-      <parent link="${prefix}link_base" />
+      <!-- <origin xyz="0.692 0.001 1.17" rpy="0 1.5708 0"    This was causing the confusion because it was linked to base now it is world />
+      <parent link="${prefix}link_base" /> -->
+      <origin xyz="0.2 -1.5 1.13" rpy="-0.0 -0.15 1.5" />
+      <parent link="world" />
       <child link="${prefix}link_camera" />
     </joint>
@@ -68,8 +70,8 @@
             <alwaysOn>true</alwaysOn>
             <updateRate>0.0</updateRate>
-            <cameraName>/camera</cameraName>
+            <cameraName>/xarm_exterior_camera</cameraName>
             <imageTopicName>image_raw</imageTopicName>
             <cameraInfoTopicName>camera_info</cameraInfoTopicName>
-            <frameName>camera_link</frameName>
+            <frameName>${prefix}link_camera</frameName>
             <hackBaseline>0.07</hackBaseline>
             <distortionK1>0.0</distortionK1>

File: xarm_ros_code/xarm_ros/xarm_description/urdf/xarm_device.urdf.xacro (robot description, xacro)
@@ -17,7 +17,7 @@
   <xacro:arg name="ros2_control_plugin" default="uf_robot_hardware/UFRobotSystemHardware"/>
   <xacro:arg name="ros2_control_params" default=""/>
-  <xacro:arg name="add_realsense_d435i" default="false"/>
+  <xacro:arg name="add_realsense_d435i" default="true"/>
   <xacro:arg name="add_d435i_links" default="true"/>
-  <xacro:arg name="use_gazebo_camera" default="false"/>
+  <xacro:arg name="use_gazebo_camera" default="true"/>
   <xacro:arg name="add_other_geometry" default="false"/>
   <xacro:arg name="geometry_type" default="box"/>

Commit message: camera position and encoding corrected

File: xarm_ros_code/xarm_ros/xarm_description/urdf/camera/camera.gazebo.xacro (robot description, xacro)
@@ -25,7 +25,5 @@
     </link>
     <joint name="${prefix}joint_camera" type="fixed">
-      <!-- <origin xyz="0.692 0.001 1.17" rpy="0 1.5708 0"    This was causing the confusion because it was linked to base now it is world />
-      <parent link="${prefix}link_base" /> -->
-      <origin xyz="0.2 -1.5 1.13" rpy="-0.0 -0.15 1.5" />
+      <origin xyz="0.8 -0.3 0.5" rpy="3.14159 2.8 0" />
       <parent link="world" />
       <child link="${prefix}link_camera" />
